Commit message: Update Assignment_1.urdf

File: Assignment_1.urdf (robot description, URDF)
Before this commit: robot Assignment_1, 4 links, 3 joints
Links:
- added link end_effector; collision box size=0.15 0.15 0.15; visual box size=0.1 0.1 0
- link arm_piece_1: geometry collision box size=0.1 0.1 1; visual box size=0.1 0.1 1
Joints:
- added joint arm_piece_3_to_end_effector: type fixed, parent arm_piece_3, child end_effector, origin xyz=0 0 0.65 rpy=0 0 0
- joint arm_piece_1_to_2: limit lower=0 upper=0 effort=0 velocity=1.0 -> lower=0 upper=6.283 effort=1000 velocity=0
- joint arm_piece_2_to_3: limit lower=0 upper=0 effort=0 velocity=1.0 -> lower=0 upper=6.283 effort=1000 velocity=0

Commit message: Update Assignment_1.urdf

File: Assignment_1.urdf (robot description, URDF)
Before this commit: robot Assignment_1, 5 links, 4 joints
Links:
- link arm_piece_2: geometry collision box size=0.1 0.1 0.9; visual box size=0.1 0.1 0.9
- link end_effector: geometry collision box size=0.1 0.1 0; visual box size=0.1 0.1 0
Joints:
- joint arm_piece_2_to_3: origin xyz=0 0 0.7 rpy=0 0 0 -> xyz=0 0 0.8 rpy=0 0 0
